File: hardware/board/butns-frontend.kicad_sch (KiCad schematic)
At the start: 262 parts, among them J1 Conn_01x08, SW1 SW_Push, SW10 SW_Push, SW11 SW_Push, SW12 SW_Push, SW13 SW_Push, SW14 SW_Push, SW15 SW_Push, SW16 SW_Push, SW17 SW_Push, SW18 SW_Push, SW19 SW_Push, SW2 SW_Push, SW20 SW_Push, SW21 SW_Push, SW22 SW_Push, SW23 SW_Push, SW24 SW_Push, SW25 SW_Push, SW26 SW_Push, SW27 SW_Push, SW28 SW_Push, SW29 SW_Push, SW3 SW_Push, SW30 SW_Push, SW31 SW_Push, SW32 SW_Push, SW33 SW_Push, SW34 SW_Push, SW35 SW_Push, SW36 SW_Push, SW37 SW_Push, SW38 SW_Push, SW39 SW_Push, SW4 SW_Push, SW40 SW_Push, SW41 SW_Push, SW42 SW_Push, SW43 SW_Push, SW44 SW_Push, SW45 SW_Push, SW46 SW_Push, SW47 SW_Push, SW48 SW_Push, SW49 SW_Push, SW5 SW_Push, SW50 SW_Push, SW51 SW_Push, SW52 SW_Push, SW53 SW_Push, SW54 SW_Push, SW55 SW_Push, SW56 SW_Push, SW57 SW_Push, SW58 SW_Push, SW59 SW_Push, SW6 SW_Push, SW60 SW_Push, SW61 SW_Push, SW62 SW_Push, SW63 SW_Push, SW64 SW_Push, SW7 SW_Push, SW8 SW_Push, SW9 SW_Push

Commit message: Convert to 16x8 grid (8 rows x 16 columns)
Hardware
- PCB extended to 190.44 x 99 mm with eight additional columns:
  128 switches, 128 diodes, 128 SK6812-EC20, 129 capacitors
- New column nets SW_COL_8..15 on GPIO16-22 and GPIO26, former
  SW_COL_8 (GPIO15) is now SW_COL_16
- LED chain runs row by row over 16 columns
- Tilt header J1 and I2C nets removed, GPIO27 left free
- Second inner mounting hole H6
- Schematic: new sheet butns-frontend2 with the 64 added cells,
  frontend and backend sheets adapted
- Regenerated jlcpcb/ gerbers, BOM and CPL, new butns.step,
  removed stale 8x8 butns.stl and model/butns.wrl

Firmware
- 16 column matrix scan per column with settle time
- LED index row * 16 + col, rotation limited to 0 and 180 degrees
- LED current estimate limited to MAX_LED_CURRENT_MA
- MPU6050 tilt support removed
- Fix led/level/row and led/level/col offset handling

Case
- case.scad and buttons.scad extended to 16 columns, second standoff
- Explicit apply_to argument for roundedcube calls

Co-Authored-By: Claude Opus 5.5 <noreply@anthropic.com>
Claude-Session: https://claude.ai/code/session_0195H63MEXeeVZ7CNyHAeb6N
Parts:
- removed J1: Conn_01x08, Connector_PinHeader_2.54mm:PinHeader_1x08_P2.54mm_Vertical_SMD_Pin1Left, symbol Connector_Generic:Conn_01x08
Connections:
- net LED_R7_A: now reaches D119.2 (DOUT)
- net LED_R7_A: no longer D120.4 (DIN)
- net LED_R3_A: now reaches D87.2 (DOUT)
- net LED_R3_A: no longer D88.4 (DIN)
- net LED_R1_A: now reaches D71.2 (DOUT)
- net LED_R1_A: no longer D72.4 (DIN)
- net LED_R4_A: now reaches D95.2 (DOUT)
- net LED_R4_A: no longer D96.4 (DIN)
- net LED_R5_A: now reaches D103.2 (DOUT)
- net LED_R5_A: no longer D104.4 (DIN)
- net LED_R6_A: now reaches D111.2 (DOUT)
- net LED_R6_A: no longer D112.4 (DIN)
- net LED_R2_A: now reaches D79.2 (DOUT)
- net LED_R2_A: no longer D80.4 (DIN)
- net LED_R8_A: now reaches D127.2 (DOUT)
- net LED_R8_A: no longer D128.4 (DIN)
- net SW_COL_8 renamed SW_COL_16
- new net LED_R1_B: D72.4 (DIN)
- new net LED_R2_B: D80.4 (DIN)
- new net LED_R3_B: D88.4 (DIN)
- new net LED_R4_B: D96.4 (DIN)
- new net LED_R5_B: D104.4 (DIN)
- new net LED_R6_B: D112.4 (DIN)
- new net LED_R7_B: D120.4 (DIN)
- new net LED_R8_B: D128.4 (DIN)
- no-connect marks 4 -> 0
